Commit message: Edit collision

File: raspimouse_description/urdf/body/body.urdf.xacro (robot description, xacro)
@@ -6,5 +6,5 @@
   <xacro:macro name="base" params="parent *joint_origin">
     <joint name="base_joint" type="fixed">
-      <insert_block name="joint_origin"/>
+      <xacro:insert_block name="joint_origin"/>
       <parent link="${parent}"/>
       <child link="base_link"/>

File: raspimouse_description/urdf/body/body_realsense.urdf.xacro (robot description, xacro)
@@ -6,5 +6,5 @@
   <xacro:macro name="base" params="parent *joint_origin">
     <joint name="base_joint" type="fixed">
-      <insert_block name="joint_origin"/>
+      <xacro:insert_block name="joint_origin"/>
       <parent link="${parent}"/>
       <child link="base_link"/>

File: raspimouse_description/urdf/body/body_urg.urdf.xacro (robot description, xacro)
@@ -6,5 +6,5 @@
   <xacro:macro name="base" params="parent *joint_origin">
     <joint name="base_joint" type="fixed">
-      <insert_block name="joint_origin"/>
+      <xacro:insert_block name="joint_origin"/>
       <parent link="${parent}"/>
       <child link="base_link"/>

File: raspimouse_description/urdf/sensors/lightsens.urdf.xacro (robot description, xacro)
@@ -4,5 +4,5 @@
   <xacro:macro name="light_sensor" params="prefix parent *joint_origin">
     <joint name="${prefix}_joint" type="fixed">
-      <insert_block name="joint_origin"/>
+      <xacro:insert_block name="joint_origin"/>
       <parent link="${parent}"/>
       <child link="${prefix}"/>

File: raspimouse_description/urdf/sensors/lrf.urdf.xacro (robot description, xacro)
@@ -4,5 +4,5 @@
   <xacro:macro name="lrf_sensor" params="prefix parent *joint_origin">
     <joint name="${prefix}_joint" type="fixed">
-      <insert_block name="joint_origin"/>
+      <xacro:insert_block name="joint_origin"/>
       <parent link="${parent}"/>
       <child link="${prefix}"/>

File: raspimouse_description/urdf/sensors/realsense.urdf.xacro (robot description, xacro)
@@ -4,5 +4,5 @@
   <xacro:macro name="rgbd_sensor" params="prefix parent *joint_origin">
     <joint name="${prefix}_joint" type="fixed">
-      <insert_block name="joint_origin"/>
+      <xacro:insert_block name="joint_origin"/>
       <parent link="${parent}"/>
       <child link="${prefix}"/>

File: raspimouse_description/urdf/wheel/wheel.urdf.xacro (robot description, xacro)
@@ -3,12 +3,12 @@
   <xacro:include filename="$(find raspimouse_description)/urdf/wheel/wheel.transmission.xacro"/>
   <xacro:include filename="$(find raspimouse_description)/urdf/wheel/wheel.gazebo.xacro"/>
-  <!-- <property name="wheel_radius" value="0.0239"/> -->
-  <property name="wheel_radius" value="0.0249"/>
-  <property name="wheel_length" value="0.01"/>
-  <property name="wheel_mass" value="0.0113"/>
+  <!-- <xacro:property name="wheel_radius" value="0.0239"/> -->
+  <xacro:property name="wheel_radius" value="0.0249"/>
+  <xacro:property name="wheel_length" value="0.01"/>
+  <xacro:property name="wheel_mass" value="0.0113"/>
   <xacro:macro name="wheel" params="prefix parent *joint_origin *joint_axis">
   <joint name="${prefix}_wheel_joint" type="continuous">
-    <insert_block name="joint_origin"/>
-    <insert_block name="joint_axis"/>
+    <xacro:insert_block name="joint_origin"/>
+    <xacro:insert_block name="joint_axis"/>
     <parent link="${parent}"/>
     <child link="${prefix}_wheel"/>
@@ -24,8 +24,8 @@
     </visual>
     <collision>
-      <!-- <insert_block name="joint_origin"/> -->
+      <!-- <xacro:insert_block name="joint_origin"/> -->
         <geometry>
-          <!-- <cylinder radius="${wheel_radius}" length="${wheel_length}"/> -->
-          <mesh filename="package://raspimouse_description/meshes/dae/wheel/RasPiMouse_wheel.dae"/>
+          <cylinder radius="${wheel_radius}" length="${wheel_length}"/>
+          <!--<mesh filename="package://raspimouse_description/meshes/dae/wheel/RasPiMouse_wheel.dae"/>-->
         </geometry>
     </collision>
