Commit message: Delete descrition for gazebo

File: raspimouse_description/urdf/raspimouse_realsense.urdf.xacro (robot description, xacro)
@@ -1,12 +1,8 @@
 <?xml version="1.0"?>
-<robot name="raspimouse_on_gazebo"
-       xmlns:sensor="http://playerstage.sourceforge.net/gazebo/xmlschema/#sensor"
-       xmlns:controller="http://playerstage.sourceforge.net/gazebo/xmlschema/#controller"
-       xmlns:interface="http://playerstage.sourceforge.net/gazebo/xmlschema/#interface"
+<robot name="raspimouse_sim"
        xmlns:xacro="http://ros.org/wiki/xacro">
   <xacro:include filename="$(find raspimouse_description)/urdf/body/body_realsense.urdf.xacro"/>
   <xacro:include filename="$(find raspimouse_description)/urdf/wheel/wheel.urdf.xacro"/>
   <xacro:include filename="$(find raspimouse_description)/urdf/sensors/lightsens.urdf.xacro"/>
-  <xacro:include filename="$(find raspimouse_description)/urdf/sensors/realsense.urdf.xacro"/>
   <!-- =============== Link & Joint =============== -->
   <!-- Base -->
@@ -37,28 +33,4 @@
     <origin xyz="0.04 0.045 0.032" rpy="0 0 0"/>
   </xacro:light_sensor>
-  <xacro:rgbd_sensor prefix="realsense_link" parent="base_link">
-    <origin xyz="0.0957 0.0175 0.0658" rpy="0 0 0"/>
-  </xacro:rgbd_sensor>
-  <!-- ===============  Transmission =============== -->
-  <!-- <xacro:wheel_trans prefix="right" interface="EffortJointInterface"/> -->
-  <!-- <xacro:wheel_trans prefix="left" interface="EffortJointInterface"/> -->
-  <xacro:wheel_trans prefix="right" interface="VelocityJointInterface"/>
-  <xacro:wheel_trans prefix="left" interface="VelocityJointInterface"/>
-  <!-- =============== Gazebo =============== -->
-  <gazebo>
-    <plugin name="gazebo_ros_control" filename="libgazebo_ros_control.so">
-      <robotNamespace>raspimouse_on_gazebo</robotNamespace>
-    </plugin>
-  </gazebo>
-  <!-- Base -->
-  <xacro:base_gazebo/>
-  <!-- Wheel -->
-  <xacro:wheel_gazebo prefix="right"/>
-  <xacro:wheel_gazebo prefix="left"/>
-  <!-- Sensors -->
-  <xacro:lightsensor_gazebo prefix="rf" base_rad="0" rad_range="0.3" min_range="0.01" max_range="0.6"/>
-  <xacro:lightsensor_gazebo prefix="rs" base_rad="-1.04" rad_range="0.3" min_range="0.01" max_range="0.6"/>
-  <xacro:lightsensor_gazebo prefix="ls" base_rad="1.04" rad_range="0.3" min_range="0.01" max_range="0.6"/>
-  <xacro:lightsensor_gazebo prefix="lf" base_rad="0" rad_range="0.3" min_range="0.01" max_range="0.6"/>
-  <raspimouse_on_gazebo/>
+  <raspimouse_sim/>
 </robot>

File: raspimouse_description/urdf/sensors/lightsens.urdf.xacro (robot description, xacro)
@@ -25,6 +25,4 @@
       </inertial>
     </link>
-    <!-- Set up laser gazebo details -->
-    <hokuyo_laser />
   </xacro:macro>
 </robot>
